Commit message: Changed the lower limit of the shoulder joint to 0 - Prevent solver from selecting non-recoverable joint configurations that require homing to recover

File: src/ik_solver/config/arm5dof.urdf (robot description, URDF)
Before this commit: robot arm5dof, 7 links, 6 joints
Joints:
- joint dof_joint03: limit lower=-2.356 upper=2.356 effort=1 velocity=1 -> lower=0.0 upper=2.356 effort=1 velocity=1
